File: test/test.kicad_sch (KiCad schematic)
At the start: 3 parts, among them J1 Barrel_Jack_MountingPin

Commit message: Add raytraced image output (#4)
* added rendering

* added rendering to test

* debug time

* fix image output path

* more debugging

* make image folder relative to project folder

* remove debugging output

* set entrypoint to fail more eagerly

* freeze kicad version for stability

As it turns out kicad nightly breaks sometimes, so freezing it prevents
that. Really we should be using stable, but 3d-rendering won't be
stable for a few months

* Fix kicad version to something that actually works

* export 3d model

* fix typos

* moved to a different branch so I can quash this later

* debugging the test which fails for some reason

* BOM generation is broken for some reason. time to wait a few months for that I guess.

* add option to set flags to adjust model size

* Kicad 9.0 has released. Need to merge back upstream eventually.

* updated test so that it doesn't fail

* clean up some stuff for upstream merge.

* fix dockerimage to use valid image
Changed lines of the file:
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@@
 (kicad_sch
-	(version 20231120)
+	(version 20250114)
 	(generator "eeschema")
-	(generator_version "8.0")
+	(generator_version "9.0")
 	(paper "A4")
 	(junction
@@
 			)
 		)
+		(property "Sim.Pins" "1=K 2=A"
+			(at 158.75 101.6 0)
+			(effects
+				(font
+					(size 1.27 1.27)
+				)
+				(hide yes)
+			)
+		)
 		(pin "1"
 		)
@@
 		)
 	)
+	(embedded_fonts no)
 )
